Commit message: Funcionando todo correctamente, comenzaré ahora a modificar para añadir cámara en la simulacion

File: TFGwebots_ws/install/tb4_sim/share/tb4_sim/resource/helper.xacro (robot description, xacro)
@@ -1,56 +1 @@
-<?xml version="1.0"?>
-<robot xmlns:xacro="http://www.ros.org/wiki/xacro" >
-    <!-- This file is not a robot in and of itself, it just contains some useful tags that could be included in any robot -->
-    <!-- Specify some colours -->
-    <material name="white">
-        <color rgba="1 1 1 1"/>
-    </material>
-    <material name="orange">
-        <color rgba="1 0.3 0.1 1"/>
-    </material>
-    <material name="blue">
-        <color rgba="0.2 0.2 1 1"/>
-    </material>
-    <material name="green">
-        <color rgba="0.2 1 0.2 1"/>
-    </material>
-    <!-- Specify some standard inertial calculations https://en.wikipedia.org/wiki/List_of_moments_of_inertia -->
-    <!-- These make use of xacro's mathematical functionality -->
-    <xacro:macro name="inertial_sphere" params="mass radius *origin">
-        <inertial>
-            <xacro:insert_block name="origin"/>
-            <mass value="${mass}" />
-            <inertia ixx="${(2/5) * mass * (radius*radius)}" ixy="0.0" ixz="0.0"
-                    iyy="${(2/5) * mass * (radius*radius)}" iyz="0.0"
-                    izz="${(2/5) * mass * (radius*radius)}" />
-        </inertial>
-    </xacro:macro>
-    <xacro:macro name="inertial_box" params="mass x y z *origin">
-        <inertial>
-            <xacro:insert_block name="origin"/>
-            <mass value="${mass}" />
-            <inertia ixx="${(1/12) * mass * (y*y+z*z)}" ixy="0.0" ixz="0.0"
-                    iyy="${(1/12) * mass * (x*x+z*z)}" iyz="0.0"
-                    izz="${(1/12) * mass * (x*x+y*y)}" />
-        </inertial>
-    </xacro:macro>
-    <xacro:macro name="inertial_cylinder" params="mass length radius *origin">
-        <inertial>
-            <xacro:insert_block name="origin"/>
-            <mass value="${mass}" />
-            <inertia ixx="${(1/12) * mass * (3*radius*radius + length*length)}" ixy="0.0" ixz="0.0"
-                    iyy="${(1/12) * mass * (3*radius*radius + length*length)}" iyz="0.0"
-                    izz="${(1/2) * mass * (radius*radius)}" />
-        </inertial>
-    </xacro:macro>
-    <!-- This is the inertial matrix of the barrier -->
-    <xacro:macro name="slender_rod" params="mass length radius *origin">
-        <inertial>
-            <xacro:insert_block name="origin"/>
-            <mass value="${mass}" />
-            <inertia ixx="${((1/3) * mass * length*length)}" ixy="0.0" ixz="0.0"
-                    iyy="0.0" iyz="0.0"
-                    izz="${((1/3) * mass * length*length)}" />
-        </inertial>
-    </xacro:macro>
-</robot>
+/home/echedey/Desktop/TFG/TFGwebots_ws/build/tb4_sim/resource/helper.xacro

File: TFGwebots_ws/install/tb4_sim/share/tb4_sim/resource/tb4_webots.xacro (robot description, xacro)
@@ -1,46 +1 @@
-<?xml version="1.0"?>
-<robot xmlns:xacro="http://wiki.ros.org/xacro">
-    <!-- tb4 robot -->
-    <xacro:include filename="$(find tb4_sim)/resource/tb4_raw.urdf" />
-    <webots>
-      <!-- Add scan config -->
-      <device reference="rplidar">
-        <ros>
-          <topicName>/scan</topicName>
-          <alwaysOn>true</alwaysOn>
-          <updateRate>20</updateRate>
-        </ros>
-      </device>
-      <plugin type="webots_ros2_driver::Ros2IMU">
-        <enabled>true</enabled>
-        <updateRate>50</updateRate>
-        <topicName>/imu</topicName>
-        <alwaysOn>true</alwaysOn>
-        <frameName>imu_link</frameName>
-        <inertialUnitName>p3d inertial</inertialUnitName>
-        <gyroName>p3d gyro</gyroName>
-      </plugin>
-      <plugin type="webots_ros2_control::Ros2Control" />
-    </webots>
-    <ros2_control name="WebotsControl" type="system">
-      <hardware>
-        <plugin>webots_ros2_control::Ros2ControlSystem</plugin>
-      </hardware>
-      <joint name="right_wheel_joint">
-        <command_interface name="velocity">
-            <param name="min">-20</param>
-            <param name="max">20</param>
-        </command_interface>
-        <state_interface name="position" />
-        <state_interface name="velocity" />
-      </joint>
-      <joint name="left_wheel_joint">
-        <command_interface name="velocity">
-            <param name="min">-20</param>
-            <param name="max">20</param>
-        </command_interface>
-        <state_interface name="position" />
-        <state_interface name="velocity" />
-      </joint>
-    </ros2_control>
-</robot>
+/home/echedey/Desktop/TFG/TFGwebots_ws/build/tb4_sim/resource/tb4_webots.xacro

File: TFGwebots_ws/src/tb4_sim/resource/tb4_webots.xacro (robot description, xacro)
@@ -1,46 +1,70 @@
 <?xml version="1.0"?>
-<robot xmlns:xacro="http://wiki.ros.org/xacro">
-    <!-- tb4 robot -->
-    <xacro:include filename="$(find tb4_sim)/resource/tb4_raw.urdf" />
-    <webots>
-      <!-- Add scan config -->
-      <device reference="rplidar">
-        <ros>
-          <topicName>/scan</topicName>
-          <alwaysOn>true</alwaysOn>
-          <updateRate>20</updateRate>
-        </ros>
-      </device>
-      <plugin type="webots_ros2_driver::Ros2IMU">
-        <enabled>true</enabled>
-        <updateRate>50</updateRate>
-        <topicName>/imu</topicName>
+<robot xmlns:xacro="http://wiki.ros.org/xacro"
+       xmlns:webots="http://www.cyberbotics.com/xacro/webots">
+  <!-- Incluir URDF crudo del TB4 -->
+  <xacro:include filename="$(find tb4_sim)/resource/tb4_raw.urdf" />
+  <webots>
+    <!-- Definición de sensores Webots dentro del robot -->
+    <webots:children>
+      <!-- Cámara virtual frontal -->
+      <!-- <webots:Camera name="camera"-->
+                     <!-- width="640" height="480"
+                     fieldOfView="1.047"   ≃60°
+                     near="0.1" far="10"
+                     translation="0 0 0.25"   ajusta altura
+                     rotation="0 1 0 0">    orientada al frente
+      </webots:Camera>  -->
+      <!-- LiDAR RPLIDAR ya definido en tb4_raw.urdf, se mapea más abajo -->
+    </webots:children>
+    <!-- Mapeo ROS para la cámara virtual -->
+    <device reference="camera">
+      <ros>
+        <topicName>/camera/image_raw</topicName>
+        <frameName>camera_link</frameName>
         <alwaysOn>true</alwaysOn>
-        <frameName>imu_link</frameName>
-        <inertialUnitName>p3d inertial</inertialUnitName>
-        <gyroName>p3d gyro</gyroName>
-      </plugin>
-      <plugin type="webots_ros2_control::Ros2Control" />
-    </webots>
-    <ros2_control name="WebotsControl" type="system">
-      <hardware>
-        <plugin>webots_ros2_control::Ros2ControlSystem</plugin>
-      </hardware>
-      <joint name="right_wheel_joint">
-        <command_interface name="velocity">
-            <param name="min">-20</param>
-            <param name="max">20</param>
-        </command_interface>
-        <state_interface name="position" />
-        <state_interface name="velocity" />
-      </joint>
-      <joint name="left_wheel_joint">
-        <command_interface name="velocity">
-            <param name="min">-20</param>
-            <param name="max">20</param>
-        </command_interface>
-        <state_interface name="position" />
-        <state_interface name="velocity" />
-      </joint>
-    </ros2_control>
+        <updateRate>30</updateRate>
+      </ros>
+    </device>
+    <!-- Mapeo ROS para el LiDAR existente -->
+    <device reference="rplidar">
+      <ros>
+        <topicName>/scan</topicName>
+        <alwaysOn>true</alwaysOn>
+        <updateRate>20</updateRate>
+      </ros>
+    </device>
+    <!-- IMU plugin -->
+    <plugin type="webots_ros2_driver::Ros2IMU">
+      <enabled>true</enabled>
+      <updateRate>50</updateRate>
+      <topicName>/imu</topicName>
+      <alwaysOn>true</alwaysOn>
+      <frameName>imu_link</frameName>
+      <inertialUnitName>p3d inertial</inertialUnitName>
+      <gyroName>p3d gyro</gyroName>
+    </plugin>
+    <!-- Control plugin -->
+    <plugin type="webots_ros2_control::Ros2Control" />
+  </webots>
+  <ros2_control name="WebotsControl" type="system">
+    <hardware>
+      <plugin>webots_ros2_control::Ros2ControlSystem</plugin>
+    </hardware>
+    <joint name="right_wheel_joint">
+      <command_interface name="velocity">
+        <param name="min">-20</param>
+        <param name="max">20</param>
+      </command_interface>
+      <state_interface name="position" />
+      <state_interface name="velocity" />
+    </joint>
+    <joint name="left_wheel_joint">
+      <command_interface name="velocity">
+        <param name="min">-20</param>
+        <param name="max">20</param>
+      </command_interface>
+      <state_interface name="position" />
+      <state_interface name="velocity" />
+    </joint>
+  </ros2_control>
 </robot>
